File: KiCAD/SN76489 arduino nano shield/SN76849 Arduino nano shield.kicad_pcb (KiCad board)
At the start: 2 copper layers, 57.4 x 43.4 mm, 10 parts, among them J2 audio_debug, J3 OLED_wit, J4 ESP32Conn, J5 LOGO, J8 geluid_uit, U1 PCF8574, U2 LM386, U3 SN76489

Commit message: Bijgewerkt
Other:
- board text added: "SN76489 ESP32 retro synth v20231106 1.0 Ontwerp: 2023 Michiel Erasmus"
- board text removed: "SN76489 Arduino retro synth v20231106 1.0 Ontwerp: 2023 Michiel Erasmus"
Changed lines of the file:
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@@
   (gr_line (start 84.1 61) (end 80.1 64)
     (stroke (width 0.15) (type default)) (layer "Edge.Cuts"))
-  (gr_text "SN76489 Arduino retro synth v20231106 1.0\nOntwerp: 2023 Michiel Erasmus" (at 60 47.4) (layer "F.SilkS")
+  (gr_text "SN76489 ESP32 retro synth v20231106 1.0\nOntwerp: 2023 Michiel Erasmus" (at 58.7 45.9) (layer "F.SilkS")
     (effects (font (size 0.7 0.7) (thickness 0.175)) (justify left))
   )

Commit message: bijgewerkt2
Parts:
- removed J8: geluid_uit, Connector_Audio:Jack_3.5mm_Lumberg_1503_07_Horizontal
- added P1: TRS_JACK, Connector_Audio:Jack_3.5mm_CUI_SJ1-3523N_Horizontal, F.Cu at (70.7, 57.4)
- C2: footprint Capacitor_THT:CP_Radial_D12.5mm_P5.00mm -> Capacitor_THT:C_Disc_D3.4mm_W2.1mm_P2.50mm
- moved C2 12.7 mm to (66.9, 40.5)
- moved RV2 2.57 mm to (56.8, 29.1)
- moved U2 1.53 mm to (52.3, 34.0)
- moved U3 1.31 mm to (41.0, 23.7)
- moved J3 1.12 mm to (38.2, 55.2)
- moved J5 0.32 mm to (71.3, 32.5)
Connections:
- net /VCC renamed VCC
- J4 pad 2: /~{WE} -> //WE
- U3 pad 5: /~{WE} -> unconnected-(U3-~{WE}-Pad5)
Routing:
- net GND: track 0.00 -> 183.0 mm, vias 0 -> 1
- net VCC: track 0.00 -> 101.9 mm, vias 0 -> 1
- net /P3: track 0.00 -> 91.6 mm, vias 0 -> 2
- net /Audio: track 0.00 -> 84.8 mm, vias 0 -> 1
- net /P4: track 0.00 -> 63.6 mm, vias 0 -> 2
- net /P0: track 0.00 -> 61.8 mm, vias 0 -> 3
- net /P2: track 0.00 -> 49.3 mm, vias 0 -> 1
- net /P1: track 0.00 -> 40.5 mm, vias 0 -> 2
- net /SDA: track 0.00 -> 40.5 mm, vias 0 -> 1
- net /SCL: track 0.00 -> 35.9 mm
- net /Clock: track 0.00 -> 33.9 mm
- net //WE: track 0.00 -> 28.2 mm, vias 0 -> 1
- net /P5: track 0.00 -> 16.9 mm
- net Net-(U2-+): track 0.00 -> 14.7 mm
- net /P6: track 0.00 -> 13.6 mm, vias 0 -> 1
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Other:
- board text added: "0,2000 mm / 0,0000 mm"
- board text added: "0,3000 mm"
- board text added: "1,6000 mm"
- board text added: "2"
- board text added: "57,5500 mm x 43,5500 mm"
- board text added: "BOARD CHARACTERISTICS"
- board text added: "Board Thickness:"
- board text added: "Board overall dimensions:"
- board text added: "Castellated pads:"
- board text added: "Copper Finish:"
- board text added: "Copper Layer Count:"
- board text added: "Edge card connectors:"
- board text added: "Impedance Control:"
- board text added: "Min hole diameter:"
- board text added: "Min track/spacing:"
- board text added: "No"
- board text added: "None"
- board text added: "Plated Board Edge:"

Commit message: PCB gerbers naar jlcpcb.com
Connections:
- U3 pad 6: GND -> unconnected-(U3-~{OE}-Pad6)
Changed lines of the file:
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@@
   (net 24 "unconnected-(U3-~{WE}-Pad5)")
   (net 25 "Net-(P1-R)")
+  (net 26 "unconnected-(U3-~{OE}-Pad6)")
   (footprint "lib_michiel:Sovjet_simpits_logo01" (layer "F.Cu")
     (at 71.3 32.5)
@@
         (effects (font (size 1 1) (thickness 0.15)))
     )
-    (fp_text value "audio_debug" (at 0 7.41) (layer "F.Fab")
+    (fp_text value "audio_debug" (at -1.27 2.8575 90) (layer "F.Fab")
         (effects (font (size 1 1) (thickness 0.15)))
     )
@@
       (net 24 "unconnected-(U3-~{WE}-Pad5)") (pinfunction "~{WE}") (pintype "power_in"))
     (pad "6" thru_hole oval (at 0 12.7) (size 1.6 1.6) (drill 0.8) (layers "*.Cu" "*.Mask")
-      (net 4 "GND") (pinfunction "~{OE}") (pintype "power_in"))
+      (net 26 "unconnected-(U3-~{OE}-Pad6)") (pinfunction "~{OE}") (pintype "power_in"))
     (pad "7" thru_hole oval (at 0 15.24) (size 1.6 1.6) (drill 0.8) (layers "*.Cu" "*.Mask")
       (net 1 "/Audio") (pinfunction "AUDIO_OUT") (pintype "input"))
