File: KiCAD/SN76489 arduino nano shield/SN76849 Arduino nano shield.kicad_sch (KiCad schematic)
At the start: 13 parts, among them J2 audio_debug, J3 OLED_wit, J4 ESP32Conn, J5 LOGO, J6 gat1, J7 gat2, J8 geluid_uit, U1 PCF8574, U3 SN76489

Commit message: Bijgewerkt
Parts:
- removed C1: CP_220uF, Capacitors_THT:CP_Radial_D10.0mm_P3.50mm, symbol SN76849 Arduino nano shield-rescue:CP1_Small-Device
- removed D1: Liggie, LEDs:LED_D3.0mm, symbol Device:LED_Small
- removed R3: R1k, w_pth_resistors:RC03, symbol Device:R_Small
- removed RV1: POT_50k, w_pth_resistors:trimmer_ecp_ca9-h2,5, symbol SN76849-Arduino-nano-shield-rescue:POT-RESCUE-SN76849_Arduino_nano_shield
- added C2: 250uF, symbol Device:C_Small
- added RV2: Pot_10k, symbol Device:R_Potentiometer_Small
- added U2: LM386, Package_DIP:DIP-8_W7.62mm, symbol Amplifier_Audio:LM386
- J4: footprint (none) -> Connector_PinHeader_2.54mm:PinHeader_1x06_P2.54mm_Vertical
Connections:
- net Audio: now also RV2.1
- net GND: now also RV2.3, U2.2 (-), U2.4 (GND)
- net VCC: now also U2.6 (V+)
- net at J8.2, J8.3, J8.4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: now also C2.2
- new net: RV2.2, U2.3 (+)
- new net: C2.1, U2.5
- no-connect marks 7 -> 9
Other:
- note added: "SN76849 WE --> ESP32 D8 SN76489 CLOCK --> ESP32 D3"
- note removed: "SN76849 WE --> Arduino D8 SN76489 CLOCK --> Arduino Nano D3"
- moved on the sheet: J2, J8

Commit message: Bijgewerkt
Parts:
- C2: footprint (none) -> Capacitor_THT:CP_Radial_D12.5mm_P5.00mm
- RV2: footprint (none) -> Potentiometer_THT:Potentiometer_Bourns_3339P_Vertical
Changed lines of the file:
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@@
       (effects (font (size 0.77 0.77)) (justify right))
     )
-    (property "Footprint" "" (at 168.529 81.788 0)
+    (property "Footprint" "Potentiometer_THT:Potentiometer_Bourns_3339P_Vertical" (at 168.529 81.788 0)
       (effects (font (size 1.27 1.27)) hide)
     )
@@
       (effects (font (size 0.77 0.77)) (justify left))
     )
-    (property "Footprint" "" (at 195.326 88.265 0)
+    (property "Footprint" "Capacitor_THT:CP_Radial_D12.5mm_P5.00mm" (at 195.326 88.265 0)
       (effects (font (size 1.27 1.27)) hide)
     )

Commit message: bijgewerkt2
Parts:
- removed J8: geluid_uit, Connector_Audio:Jack_3.5mm_Lumberg_1503_07_Horizontal, symbol SN76849 Arduino nano shield-rescue:Audio-Jack-5-conn
- added P1: TRS_JACK, Connector_Audio:Jack_3.5mm_CUI_SJ1-3523N_Horizontal, symbol trs_jack:TRS_JACK
- C2: footprint Capacitor_THT:CP_Radial_D12.5mm_P5.00mm -> Capacitor_THT:C_Disc_D3.4mm_W2.1mm_P2.50mm
Connections:
- net GND: now also P1.1 (S); no longer U3.6 (~{OE})
- net at C2.2: now also P1.2 (T), P1.3 (R)
- net ~{WE}: no longer names the net of U3.5 (~{WE})
- net ~{WE}: no longer J4.2 (Pin_2)
- new net /WE: J4.2 (Pin_2)
Other:
- note added: "3.5mm_CUI_SJ1-3523N"
- note removed: "PJ307 3.5mm uitgang"
- moved on the sheet: C2, J2, J3, J4, RV2, U2, U3
